File: Punainen insinööri.kicad_pcb (KiCad board)
At the start: 2 copper layers, 19 parts, among them Q1 MMBFJ113, U1 LF351D

Commit message: jotain säätöä
Parts:
- added C8: 10uF, Capacitor_SMD:CP_Elec_4x5.4, F.Cu at (117.8, 55.9)
- added C9: 100uF, Capacitor_SMD:CP_Elec_6.3x5.4, F.Cu at (134.4, 45.0)
- added J1: Barrel_Jack_Switch, Connector_BarrelJack:BarrelJack_Horizontal, F.Cu at (106.9, 52.3)
- moved C1 22.4 mm to (124.3, 45.0), turned to -90 degrees

Commit message: the trans question
Parts:
- moved Q1 4.29 mm to (113.2, 68.2)
Changed lines of the file:
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@@
   (net 19 "unconnected-(J1-Pad3)")
   (footprint "Package_TO_SOT_SMD:SOT-23" (layer "F.Cu")
-    (at 108.9425 67.49)
+    (at 113.1725 68.21)
     (descr "SOT, 3 Pin (https://www.jedec.org/system/files/docs/to-236h.pdf variant AB), generated with kicad-footprint-generator ipc_gullwing_generator.py")
     (tags "SOT TO_SOT_SMD")
@@
       (stroke (width 0.1) (type solid)) (layer "F.Fab"))
     (pad "1" smd roundrect (at -2.575 -1.905) (size 1.75 0.6) (layers "F.Cu" "F.Paste" "F.Mask") (roundrect_rratio 0.25)
-      (net 5 "unconnected-(U1-NULL-Pad1)") (pinfunction "NULL") (pintype "input"))
+      (net 5 "unconnected-(U1-NULL-Pad1)") (pinfunction "NULL") (pintype "input+no_connect"))
     (pad "2" smd roundrect (at -2.575 -0.635) (size 1.75 0.6) (layers "F.Cu" "F.Paste" "F.Mask") (roundrect_rratio 0.25)
       (net 6 "Net-(LED1-K)") (pinfunction "-") (pintype "input"))
@@
       (net 2 "GND") (pinfunction "V-") (pintype "power_in"))
     (pad "5" smd roundrect (at 2.575 1.905) (size 1.75 0.6) (layers "F.Cu" "F.Paste" "F.Mask") (roundrect_rratio 0.25)
-      (net 8 "unconnected-(U1-NULL-Pad5)") (pinfunction "NULL") (pintype "input"))
+      (net 8 "unconnected-(U1-NULL-Pad5)") (pinfunction "NULL") (pintype "input+no_connect"))
     (pad "6" smd roundrect (at 2.575 0.635) (size 1.75 0.6) (layers "F.Cu" "F.Paste" "F.Mask") (roundrect_rratio 0.25)
       (net 9 "Net-(LED1-A)") (pintype "output"))

Commit message: millenials in shambles
Parts:
- added C10: 10nF, Capacitor_SMD:C_0805_2012Metric_Pad1.18x1.45mm_HandSolder, F.Cu at (93.7, 61.6)
- added D2: 1N4148W, Diode_SMD:D_SOD-123, F.Cu at (176.7, 48.2)
- added D3: 1N4148W, Diode_SMD:D_SOD-123, F.Cu at (159.8, 48.0)
- added LED1: LED_Small, LED_SMD:LED_1206_3216Metric_Pad1.42x1.75mm_HandSolder, F.Cu at (93.4, 69.7)
- added LED2: LED_Small, LED_SMD:LED_1206_3216Metric_Pad1.42x1.75mm_HandSolder, F.Cu at (93.4, 66.3)
- added Q2: MMBF170, Package_TO_SOT_SMD:SOT-23, F.Cu at (172.5, 47.5)
- added Q3: MMBF170, Package_TO_SOT_SMD:SOT-23, F.Cu at (155.7, 47.4)
- added R10: 4.7k, Resistor_SMD:R_0805_2012Metric_Pad1.20x1.40mm_HandSolder, F.Cu at (172.6, 50.8)
- added R11: 4.7k, Resistor_SMD:R_0805_2012Metric_Pad1.20x1.40mm_HandSolder, F.Cu at (155.8, 50.5)
- added REF**: Pin_D0.7mm_L6.5mm_W1.8mm_FlatFork, Connector_Pin:Pin_D0.7mm_L6.5mm_W1.8mm_FlatFork, F.Cu at (179.6, 50.8)
- added REF**: Pin_D0.7mm_L6.5mm_W1.8mm_FlatFork, Connector_Pin:Pin_D0.7mm_L6.5mm_W1.8mm_FlatFork, F.Cu at (162.8, 50.5)
- added REF**: Pin_D0.7mm_L6.5mm_W1.8mm_FlatFork, Connector_Pin:Pin_D0.7mm_L6.5mm_W1.8mm_FlatFork, F.Cu at (162.8, 46.4)
- added REF**: Pin_D0.7mm_L6.5mm_W1.8mm_FlatFork, Connector_Pin:Pin_D0.7mm_L6.5mm_W1.8mm_FlatFork, F.Cu at (179.6, 46.6)
- Q1: value MMBFJ113 -> MMBF4393LT1G
- moved C2 13.7 mm to (128.1, 55.4)
- moved C3 13.7 mm to (128.1, 58.4)
- moved C5 13.7 mm to (128.1, 64.5)
- moved C6 13.7 mm to (128.1, 67.5)
- moved R1 13.7 mm to (123.3, 55.4)
- moved R2 13.7 mm to (123.3, 58.4)
- moved R3 13.7 mm to (123.3, 61.3)
- moved R4 13.7 mm to (123.3, 64.2)
- moved R7 13.7 mm to (123.3, 73.1)
- moved R8 13.7 mm to (123.3, 76.0)
- moved C4 13.7 mm to (128.1, 61.5)
- moved C7 13.7 mm to (128.1, 70.5)
- moved R5 13.7 mm to (123.3, 67.2)
- moved R6 13.7 mm to (123.3, 70.2)
Routing:
- net +9V: track 0.00 -> 8.30 mm
- net FS_red: track 0.00 -> 7.95 mm
- net FS_engi: track 0.00 -> 7.95 mm
- net Net-(LED3-A): track 0.00 -> 5.95 mm
- net Net-(LED4-A): track 0.00 -> 5.95 mm
- net Net-(Q2-S): track 0.00 -> 2.25 mm

Commit message: Schema valmiina
Parts:
- added C11: 10nF, Capacitor_SMD:C_0805_2012Metric_Pad1.18x1.45mm_HandSolder, F.Cu at (77.2, 55.5)
- added C12: 10nF, Capacitor_SMD:C_0805_2012Metric_Pad1.18x1.45mm_HandSolder, F.Cu at (74.5, 62.0)
- added SW2: SW_DPDT_x2, Button_Switch_THT:SW_Push_2P2T_Toggle_CK_PVA2xxH1xxxxxxV2, F.Cu at (140.7, 63.7)
- added U2: TL074, Package_SO:SO-14_3.9x8.65mm_P1.27mm, F.Cu at (82.2, 56.0)
- added U3: LM13700, Package_SO:SOP-16_3.9x9.9mm_P1.27mm, F.Cu at (69.1, 61.2)

Commit message: pieniä muutoksia
Parts:
- added C13: 1uF, Capacitor_SMD:C_0805_2012Metric_Pad1.18x1.45mm_HandSolder, F.Cu at (94.8, 32.0)
- added C14: 10nF, Capacitor_SMD:C_0805_2012Metric_Pad1.18x1.45mm_HandSolder, F.Cu at (-40.8, 77.0)
- added C15: 100pF, Capacitor_SMD:C_0805_2012Metric_Pad1.18x1.45mm_HandSolder, F.Cu at (-40.8, 80.0)
- added C16: 4.7nF, Capacitor_SMD:C_0805_2012Metric_Pad1.18x1.45mm_HandSolder, F.Cu at (-40.8, 83.0)
- added C17: 10uF, Capacitor_SMD:CP_Elec_4x5.4, F.Cu at (-31.0, 98.7)
- added C18: 1uF, Capacitor_SMD:C_0805_2012Metric_Pad1.18x1.45mm_HandSolder, F.Cu at (-40.8, 86.0)
- added C19: 1uF, Capacitor_SMD:C_0805_2012Metric_Pad1.18x1.45mm_HandSolder, F.Cu at (-40.8, 89.1)
- added D4: 1N4148W, Diode_SMD:D_SOD-123, F.Cu at (-35.5, 74.2)
- added D5: 1N4148W, Diode_SMD:D_SOD-123, F.Cu at (-35.5, 77.5)
- added D6: 1N4148W, Diode_SMD:D_SOD-123, F.Cu at (-35.5, 80.9)
- added LED5: LED_Small, LED_SMD:LED_1206_3216Metric_Pad1.42x1.75mm_HandSolder, F.Cu at (-46.7, 91.9)
- added LED6: LED_Small, LED_SMD:LED_1206_3216Metric_Pad1.42x1.75mm_HandSolder, F.Cu at (-46.7, 95.3)
- added Q4: BC807, Package_TO_SOT_SMD:SOT-23, F.Cu at (-36.0, 84.8)
- added R12: 10k, Resistor_SMD:R_0805_2012Metric_Pad1.20x1.40mm_HandSolder, F.Cu at (80.5, 31.9)
- added R13: 10k, Resistor_SMD:R_0805_2012Metric_Pad1.20x1.40mm_HandSolder, F.Cu at (80.5, 34.9)
- added R14: 1M, Resistor_SMD:R_0805_2012Metric_Pad1.20x1.40mm_HandSolder, F.Cu at (80.5, 37.8)
- added R15: 1M, Resistor_SMD:R_0805_2012Metric_Pad1.20x1.40mm_HandSolder, F.Cu at (80.5, 40.8)
- added R16: 1M, Resistor_SMD:R_0805_2012Metric_Pad1.20x1.40mm_HandSolder, F.Cu at (-55.1, 85.8)
- added R17: 1k, Resistor_SMD:R_0805_2012Metric_Pad1.20x1.40mm_HandSolder, F.Cu at (-55.1, 88.7)
- added R18: 1M, Resistor_SMD:R_0805_2012Metric_Pad1.20x1.40mm_HandSolder, F.Cu at (-50.4, 74.0)
- added R19: 10k, Resistor_SMD:R_0805_2012Metric_Pad1.20x1.40mm_HandSolder, F.Cu at (-50.4, 76.9)
- added R20: 10k, Resistor_SMD:R_0805_2012Metric_Pad1.20x1.40mm_HandSolder, F.Cu at (-50.4, 79.9)
- added R21: 10k, Resistor_SMD:R_0805_2012Metric_Pad1.20x1.40mm_HandSolder, F.Cu at (-50.4, 82.8)
- added R22: 220Ω, Resistor_SMD:R_0805_2012Metric_Pad1.20x1.40mm_HandSolder, F.Cu at (-50.4, 85.8)
- added R23: 1k, Resistor_SMD:R_0805_2012Metric_Pad1.20x1.40mm_HandSolder, F.Cu at (-50.4, 88.7)
- added R24: 470k, Resistor_SMD:R_0805_2012Metric_Pad1.20x1.40mm_HandSolder, F.Cu at (-45.6, 74.0)
- added R25: 100Ω, Resistor_SMD:R_1206_3216Metric_Pad1.30x1.75mm_HandSolder, F.Cu at (-35.4, 88.6)
- added R26: 1k, Resistor_SMD:R_0805_2012Metric_Pad1.20x1.40mm_HandSolder, F.Cu at (-45.6, 76.9)
- added R27: 1M, Resistor_SMD:R_0805_2012Metric_Pad1.20x1.40mm_HandSolder, F.Cu at (-45.6, 79.9)
- added R28: 1k, Resistor_SMD:R_0805_2012Metric_Pad1.20x1.40mm_HandSolder, F.Cu at (-45.6, 82.8)
- added REF**: Pin_D1.0mm_L10.0mm, Connector_Pin:Pin_D1.0mm_L10.0mm, F.Cu at (172.0, 72.4)
- added REF**: Pin_D1.0mm_L10.0mm, Connector_Pin:Pin_D1.0mm_L10.0mm, F.Cu at (179.1, 72.4)
- added SW1: SW_DPDT_x2, Button_Switch_THT:SW_Push_2P2T_Toggle_CK_PVA2xxH1xxxxxxV2, F.Cu at (153.5, 122.5)
- added rv1: 1M, Potentiometer_THT:Potentiometer redwiz, B.Cu at (174.0, 99.1)
- added rv2: 100k, Potentiometer_THT:Potentiometer redwiz, F.Cu at (163.0, 113.3)
- added rv3: 100k, Potentiometer_THT:Potentiometer redwiz, B.Cu at (148.6, 99.1)
- added rv4: 1M, Potentiometer_THT:Potentiometer redwiz, F.Cu at (-12.3, 96.9)
- added rv5: 10k, Potentiometer_THT:Potentiometer redwiz, B.Cu at (97.8, 99.1)
- added rv6: 100k, Potentiometer_THT:Potentiometer redwiz, B.Cu at (123.2, 99.1)
- C1, C9, D1, R9: moved to B.Cu
- moved C12 151.6 mm to (-74.0, 92.4)
- moved U2 143.9 mm to (-60.0, 78.0)
- moved U3 143.9 mm to (-73.1, 83.1)
- moved C11 140.1 mm to (-59.5, 86.3)
- moved Q3 90.6 mm to (69.5, 19.5)
- moved R11 90.6 mm to (69.5, 22.7)
- moved REF** 90.6 mm to (93.3, 22.9)
- moved REF** 90.6 mm to (93.3, 18.8)
- moved D2 90.6 mm to (90.4, 20.4)
- moved D3 90.6 mm to (73.6, 20.2)
- moved Q2 90.6 mm to (86.3, 19.7)
- moved R10 90.6 mm to (86.3, 22.9)
- moved REF** 90.6 mm to (76.5, 22.7)
- moved REF** 90.6 mm to (76.5, 18.6)
- moved C10 88.3 mm to (178.7, 85.4), turned to 90 degrees
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Connections:
- U2 pad 1: unconnected-(U2-Pad1) -> +5V
- U2 pad 10: unconnected-(U2C-+-Pad10) -> Net-(U2B-+)
- U2 pad 12: unconnected-(U2D-+-Pad12) -> Net-(U2D-+)
- U2 pad 13: unconnected-(U2D---Pad13) -> Net-(D6-K)
- U2 pad 14: unconnected-(U2-Pad14) -> Net-(D6-A)
- U2 pad 2: unconnected-(U2A---Pad2) -> +5V
- U2 pad 3: unconnected-(U2A-+-Pad3) -> Net-(U2A-+)
- U2 pad 5: unconnected-(U2B-+-Pad5) -> Net-(U2B-+)
- U2 pad 6: unconnected-(U2B---Pad6) -> Net-(D4-K)
- U2 pad 7: unconnected-(U2-Pad7) -> Net-(D4-A)
- U2 pad 8: unconnected-(U2-Pad8) -> Net-(C15-Pad1)
- U2 pad 9: unconnected-(U2C---Pad9) -> Net-(U2C--)
- U3 pad 1: unconnected-(U3-Pad1) -> Net-(Q4-C)
- U3 pad 10: unconnected-(U3-Pad10) -> Net-(U3-Pad10)
- U3 pad 12: unconnected-(U3-Pad12) -> Net-(U3A--)
- U3 pad 13: unconnected-(U3A---Pad13) -> Net-(U3A--)
- U3 pad 14: unconnected-(U3A-+-Pad14) -> Net-(U3A-+)
- U3 pad 16: unconnected-(U3-Pad16) -> GND
- U3 pad 3: unconnected-(U3C-+-Pad3) -> Net-(U3C-+)
- U3 pad 4: unconnected-(U3C---Pad4) -> +5V
- U3 pad 5: unconnected-(U3-Pad5) -> Net-(U2C--)
- U3 pad 7: unconnected-(U3-Pad7) -> Net-(U3-Pad7)
- U3 pad 8: unconnected-(U3-Pad8) -> Net-(U3-Pad7)
- U3 pad 9: unconnected-(U3-Pad9) -> Net-(U3-Pad10)
Routing:
- net +9V: track 8.30 -> 60.3 mm, vias 0 -> 6
- net Net-(Q1-S): track 0.00 -> 45.8 mm
- net Net-(LED1-A): track 0.00 -> 28.8 mm, vias 0 -> 1
- net Net-(LED1-K): track 0.00 -> 26.8 mm
- net Net-(R6-Pad1): track 0.00 -> 19.9 mm
- net Net-(U1-+): track 0.00 -> 15.6 mm
- net Net-(C6-Pad1): track 0.00 -> 6.68 mm
- net Net-(C5-Pad1): track 0.00 -> 6.47 mm
- net Net-(Q1-G): track 0.00 -> 5.43 mm
- net IN_red_pcb: track 0.00 -> 5.43 mm
- net Net-(R5-Pad1): track 0.00 -> 4.85 mm
- net Net-(C8-Pad2): track 0.00 -> 3.58 mm
- net Net-(J1-Pad2): track 0.00 -> 2.96 mm
- net Net-(C4-Pad1): track 0.00 -> 2.16 mm
- net GND: vias 0 -> 4
- added copper zone on B.Cu, net GND
- added copper zone on F.Cu, net GND
Other:
- board outline added: 103.6 x 64 mm
- board text added: "+DC-"
- board text added: "-DC+"

Commit message: pcb v1
Parts:
- removed J1: Barrel_Jack_Switch, Connector_BarrelJack:BarrelJack_Horizontal
- removed SW1, SW2: SW_DPDT_x2, Button_Switch_THT:SW_Push_2P2T_Toggle_CK_PVA2xxH1xxxxxxV2
- added GND: Pin_D1.0mm_L10.0mm, Connector_Pin:Pin_D1.0mm_L10.0mm, F.Cu at (158.2, 122.2)
- added GND: Pin_D1.0mm_L10.0mm, Connector_Pin:Pin_D1.0mm_L10.0mm, F.Cu at (162.2, 122.2)
- added GND: Pin_D1.0mm_L10.0mm, Connector_Pin:Pin_D1.0mm_L10.0mm, F.Cu at (112.3, 122.2)
- added GND: Pin_D1.0mm_L10.0mm, Connector_Pin:Pin_D1.0mm_L10.0mm, F.Cu at (108.3, 122.2)
- added IN_ENGI: Pin_D1.0mm_L10.0mm, Connector_Pin:Pin_D1.0mm_L10.0mm, F.Cu at (91.0, 122.2)
- added IN_RED: Pin_D1.0mm_L10.0mm, Connector_Pin:Pin_D1.0mm_L10.0mm, F.Cu at (168.2, 122.2)
- added OUT_ENGI: Pin_D1.0mm_L10.0mm, Connector_Pin:Pin_D1.0mm_L10.0mm, F.Cu at (97.8, 122.2)
- added OUT_RED: Pin_D1.0mm_L10.0mm, Connector_Pin:Pin_D1.0mm_L10.0mm, F.Cu at (175.0, 122.2)
- C11, C12, C17, C8, rv2, rv4: moved to B.Cu
- moved U3 198.7 mm to (124.4, 104.9), turned to 90 degrees
- moved C12 198.1 mm to (123.7, 104.7), turned to 180 degrees
- moved R20 189.2 mm to (136.0, 112.7), turned to 90 degrees
- moved R19 186.1 mm to (132.3, 112.7), turned to 90 degrees
- moved R21 177.9 mm to (125.0, 112.7), turned to -90 degrees
- moved C16 177.3 mm to (133.3, 116.1)
- moved R22 173.7 mm to (121.3, 112.7), turned to 90 degrees
- moved C15 172.5 mm to (128.6, 112.7), turned to 90 degrees
- moved R27 166.6 mm to (117.7, 112.7), turned to 90 degrees
- moved U2 162.1 mm to (102.0, 83.4), turned to -90 degrees
- moved C11 160.4 mm to (100.9, 83.4), turned to 180 degrees
- moved R28 153.7 mm to (108.1, 81.9), turned to -90 degrees
- moved R23 148.6 mm to (98.2, 89.8), turned to -90 degrees
- moved R18 148.0 mm to (94.5, 104.2), turned to 90 degrees
- moved R17 147.5 mm to (91.0, 108.7), turned to 90 degrees
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Routing:
- net +9V: track 60.3 -> 185.7 mm
- net +5V: track 0.00 -> 92.7 mm, vias 0 -> 2
- net Net-(U2C--): track 0.00 -> 62.5 mm, vias 0 -> 1
- net Net-(C18-Pad1): track 0.00 -> 57.2 mm, vias 0 -> 1
- net Net-(C15-Pad1): track 0.00 -> 50.6 mm
- net OUT_red_pcb: track 0.00 -> 44.5 mm
- net Net-(R25-Pad2): track 0.00 -> 38.5 mm, vias 0 -> 1
- net IN_red_pcb: track 5.43 -> 41.3 mm
- net Net-(U2B-+): track 0.00 -> 34.7 mm
- net Net-(Q4-C): track 0.00 -> 28.9 mm
- net Net-(U2D-+): track 0.00 -> 27.4 mm, vias 0 -> 2
- net OUT_engi_pcb: track 0.00 -> 27.0 mm
- net Net-(Q1-S): track 45.8 -> 22.7 mm, vias 0 -> 1
- net IN_engi_pcb: track 0.00 -> 16.1 mm
- net Net-(C8-Pad2): track 3.58 -> 17.3 mm
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Other:
- board text added: "ENGI THUMB"
- board text added: "GND"
- board text added: "IN_ENGI"
- board text added: "IN_RED"
- board text added: "OUT_ENGI"
- board text added: "OUT_RED"
- board text added: "RED FUZZ"

Commit message: pcb v1.1
Parts:
- C1, C11, C12, C17, C8, C9, D1, R9: moved to F.Cu
- moved REF** 37.0 mm to (142.2, 74.3), turned to 180 degrees
- moved D1 33.9 mm to (142.2, 80.4)
- moved R9 22.9 mm to (149.3, 80.2)
- moved REF** 22.8 mm to (149.3, 74.3), turned to 180 degrees
- moved C8 15.5 mm to (146.6, 90.3), turned to 180 degrees
- moved C12 7.00 mm to (127.3, 98.7), turned to 0 degrees
- moved C2 6.80 mm to (163.4, 95.9)
- moved C11 6.08 mm to (101.0, 77.3)
- moved R1 5.95 mm to (163.5, 87.1), turned to 0 degrees
- moved R15 5.49 mm to (108.5, 78.3), turned to 0 degrees
- moved C10 5.23 mm to (174.9, 81.8), turned to 0 degrees
- moved R13 4.94 mm to (116.5, 98.7), turned to 180 degrees
- moved R14 4.86 mm to (104.1, 74.2)
- moved C3 4.39 mm to (156.8, 95.9)
- moved C16 3.95 mm to (136.9, 114.4)
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Routing:
- net +9V: track 185.7 -> 170.7 mm, vias 6 -> 0
- net Net-(Q1-S): track 22.7 -> 35.0 mm, vias 1 -> 2
- net Net-(C8-Pad2): track 17.3 -> 4.96 mm
- net Net-(LED5-K): track 9.77 -> 15.4 mm
- net Net-(U2B-+): track 34.7 -> 31.3 mm
- net Net-(U2C--): track 62.5 -> 59.5 mm
- net +5V: track 92.7 -> 95.7 mm
- net Net-(U2A-+): track 9.93 -> 12.4 mm
- net Net-(Q1-G): track 5.43 -> 6.89 mm
- net Net-(C16-Pad1): track 2.40 -> 3.86 mm
- net Net-(J1-Pad2): track 2.96 -> 4.40 mm
- net Net-(LED1-K): track 28.3 -> 27.0 mm
- net Net-(U3A-+): track 6.30 -> 7.47 mm
- net Net-(R5-Pad1): track 5.35 -> 4.41 mm
- net Net-(C6-Pad1): track 6.68 -> 7.48 mm
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Other:
- board size 103.6 x 64 mm -> 104 x 64.5 mm
- board text added: "+DC- 9V"
- board text added: "-DC+ 9V"
- board text added: "HARRI SIE OOT MUNAPARTAVELEHO"
- board text added: "JLCJLCJLCJLC"
- board text added: "JUHO RYTKÖNEN https://github.com/Secret624/redWizard"
- board text removed: "+DC-"
- board text removed: "-DC+"

Commit message: pcb v1.2
Parts:
- moved R7 9.72 mm to (182.3, 82.3), turned to 90 degrees
- moved C6 8.06 mm to (179.8, 103.7), turned to 180 degrees
- moved R16 7.60 mm to (92.0, 114.8), turned to 0 degrees
- moved Q1 1.15 mm to (181.4, 87.4)
Routing:
- net Net-(C6-Pad1): track 7.48 -> 11.6 mm
- net IN_engi_pcb: track 16.1 -> 12.5 mm
- net Net-(C18-Pad1): track 57.2 -> 54.7 mm
- net Net-(Q1-S): track 35.0 -> 33.5 mm
- net +9V: track 170.7 -> 169.5 mm
- net GND: vias 36 -> 32
Other:
- board size 104 x 64.5 mm -> 96 x 56.3 mm
- board text removed: "HARRI SIE OOT MUNAPARTAVELEHO"
