File: Punainen insinööri.kicad_pcb (KiCad board)
At the start: 2 copper layers, 96 x 56.3 mm, 84 parts, among them Q1 MMBF4393LT1G, Q2 MMBF170, Q3 MMBF170, Q4 BC807, U1 LF351D, U2 TL074, U3 LM13700

Commit message: Konkan tuplaus temppu
Parts:
- added C20: 10uF, Capacitor_SMD:CP_Elec_4x5.4, B.Cu at (101.6, 101.0)
- added C21: 10uF, Capacitor_SMD:CP_Elec_4x5.4, B.Cu at (146.6, 90.3)
- added C22: 100uF, Capacitor_SMD:CP_Elec_6.3x5.4, B.Cu at (156.4, 79.0)
- added C23: 100uF, Capacitor_SMD:CP_Elec_6.3x5.4, B.Cu at (165.0, 79.0)
- moved R23 1.05 mm to (98.2, 90.8)
Routing:
- net +9V: track 169.5 -> 178.1 mm, vias 0 -> 2
- net Net-(C17-Pad1): track 13.4 -> 20.0 mm, vias 0 -> 1
- net Net-(C21-Pad2): track 4.96 -> 9.92 mm
- net Net-(C17-Pad2): track 3.92 -> 7.82 mm
- net Net-(Q1-S): track 33.5 -> 37.2 mm
- net +5V: track 95.7 -> 98.1 mm
- net Net-(Q4-C): track 28.9 -> 27.1 mm
- net IN_red_pcb: track 40.6 -> 39.7 mm
- net Net-(U2C--): track 59.5 -> 58.9 mm
