File: Punainen insinööri.kicad_pcb (KiCad board)
At the start: 2 copper layers, 96 x 56.3 mm, 88 parts, among them Q1 MMBF4393LT1G, Q2 MMBF170, Q3 MMBF170, Q4 BC807, U1 LF351D, U2 TL074, U3 LM13700

Commit message: Ledin lisäys loitsu
Parts:
- added LED7: LED_Small, LED_THT:LED_D3.0mm, B.Cu at (93.2, 105.2)
- added LED8: LED_Small, LED_THT:LED_D3.0mm, F.Cu at (102.0, 112.0)
- moved LED6 1.83 mm to (98.6, 109.2)
Routing:
- net Net-(LED5-K): track 15.4 -> 17.7 mm
- net GND: vias 32 -> 30
Changed lines of the file:
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@@
     )
   )
+  (footprint "LED_THT:LED_D3.0mm" (layer "F.Cu")
+    (at 102.04 112.015 90)
+    (descr "LED, diameter 3.0mm, 2 pins")
+    (tags "LED diameter 3.0mm 2 pins")
+    (property "LCSC#" "")
+    (property "Sheetfile" "Punainen insinööri.kicad_sch")
+    (property "Sheetname" "")
+    (property "ki_description" "Light emitting diode, small symbol")
+    (property "ki_keywords" "LED diode light-emitting-diode")
+    (attr through_hole)
+    (fp_text reference "LED8" (at -1.875 0 180) (layer "F.SilkS")
+        (effects (font (size 1 1) (thickness 0.15)))
+    )
+    (fp_text value "LED_Small" (at 1.27 2.96 90) (layer "F.Fab")
+        (effects (font (size 1 1) (thickness 0.15)))
+    )
+    (fp_line (start -0.29 -1.236) (end -0.29 -1.08)
+      (stroke (width 0.12) (type solid)) (layer "F.SilkS"))
+    (fp_line (start -0.29 1.08) (end -0.29 1.236)
+      (stroke (width 0.12) (type solid)) (layer "F.SilkS"))
+    (fp_arc (start -0.29 -1.235516) (mid 1.366487 -1.987659) (end 2.942335 -1.078608)
+      (stroke (width 0.12) (type solid)) (layer "F.SilkS"))
+    (fp_arc (start 0.229039 -1.08) (mid 1.270117 -1.5) (end 2.31113 -1.079837)
+      (stroke (width 0.12) (type solid)) (layer "F.SilkS"))
+    (fp_arc (start 2.31113 1.079837) (mid 1.270117 1.5) (end 0.229039 1.08)
+      (stroke (width 0.12) (type solid)) (layer "F.SilkS"))
+    (fp_arc (start 2.942335 1.078608) (mid 1.366487 1.987659) (end -0.29 1.235516)
+      (stroke (width 0.12) (type solid)) (layer "F.SilkS"))
+    (fp_line (start -1.15 -2.25) (end -1.15 2.25)
+      (stroke (width 0.05) (type solid)) (layer "F.CrtYd"))
+    (fp_line (start -1.15 2.25) (end 3.7 2.25)
+      (stroke (width 0.05) (type solid)) (layer "F.CrtYd"))
+    (fp_line (start 3.7 -2.25) (end -1.15 -2.25)
+      (stroke (width 0.05) (type solid)) (layer "F.CrtYd"))
+    (fp_line (start 3.7 2.25) (end 3.7 -2.25)
+      (stroke (width 0.05) (type solid)) (layer "F.CrtYd"))
+    (fp_line (start -0.23 -1.16619) (end -0.23 1.16619)
+      (stroke (width 0.1) (type solid)) (layer "F.Fab"))
+    (fp_arc (start -0.23 -1.16619) (mid 3.17 0.000452) (end -0.230555 1.165476)
+      (stroke (width 0.1) (type solid)) (layer "F.Fab"))
+    (fp_circle (center 1.27 0) (end 2.77 0)
+      (stroke (width 0.1) (type solid)) (fill none) (layer "F.Fab"))
+    (pad "1" thru_hole rect (at 0 0 90) (size 1.8 1.8) (drill 0.9) (layers "*.Cu" "*.Mask")
+      (net 2 "GND") (pinfunction "K") (pintype "passive"))
+    (pad "2" thru_hole circle (at 2.54 0 90) (size 1.8 1.8) (drill 0.9) (layers "*.Cu" "*.Mask")
+      (net 29 "Net-(LED5-K)") (pinfunction "A") (pintype "passive"))
+    (model "${KICAD6_3DMODEL_DIR}/LED_THT.3dshapes/LED_D3.0mm.wrl"
+      (offset (xyz 0 0 0))
+      (scale (xyz 1 1 1))
+      (rotate (xyz 0 0 0))
+    )
+  )
   (footprint "Connector_Pin:Pin_D1.0mm_L10.0mm" (layer "F.Cu")
     (at 91 122.2)
@@
     (property "ki_keywords" "LED diode light-emitting-diode")
     (attr smd)
-    (fp_text reference "LED5" (at 3.5 0 -180) (layer "F.SilkS")
+    (fp_text reference "LED5" (at 3.35 0.79 -180) (layer "F.SilkS")
         (effects (font (size 1 1) (thickness 0.15)))
     )
@@
   )
   (footprint "LED_SMD:LED_1206_3216Metric_Pad1.42x1.75mm_HandSolder" (layer "F.Cu")
-    (at 100.4 109.2 90)
+    (at 98.57 109.21 90)
     (descr "LED SMD 1206 (3216 Metric), square (rectangular) end terminal, IPC_7351 nominal, (Body size source: http://www.tortai-tech.com/upload/download/2011102023233369053.pdf), generated with kicad-footprint-generator")
     (tags "LED handsolder")
@@
       (net 36 "Net-(C18-Pad1)") (pinfunction "3") (pintype "passive"))
   )
+  (footprint "LED_THT:LED_D3.0mm" (layer "B.Cu")
+    (at 93.25 105.175 -90)
+    (descr "LED, diameter 3.0mm, 2 pins")
+    (tags "LED diameter 3.0mm 2 pins")
+    (property "LCSC#" "C84263")
+    (property "Sheetfile" "Punainen insinööri.kicad_sch")
+    (property "Sheetname" "")
+    (property "ki_description" "Light emitting diode, small symbol")
+    (property "ki_keywords" "LED diode light-emitting-diode")
+    (attr through_hole)
+    (fp_text reference "LED7" (at 4.39 -0.01) (layer "B.SilkS")
+        (effects (font (size 1 1) (thickness 0.15)) (justify mirror))
+    )
+    (fp_text value "LED_Small" (at 1.27 -2.96 90) (layer "B.Fab")
+        (effects (font (size 1 1) (thickness 0.15)) (justify mirror))
+    )
+    (fp_line (start -0.29 -1.08) (end -0.29 -1.236)
+      (stroke (width 0.12) (type solid)) (layer "B.SilkS"))
+    (fp_line (start -0.29 1.236) (end -0.29 1.08)
+      (stroke (width 0.12) (type solid)) (layer "B.SilkS"))
+    (fp_arc (start -0.29 -1.235516) (mid 1.366487 -1.987659) (end 2.942335 -1.078608)
+      (stroke (width 0.12) (type solid)) (layer "B.SilkS"))
+    (fp_arc (start 0.229039 -1.08) (mid 1.270117 -1.5) (end 2.31113 -1.079837)
+      (stroke (width 0.12) (type solid)) (layer "B.SilkS"))
+    (fp_arc (start 2.31113 1.079837) (mid 1.270117 1.5) (end 0.229039 1.08)
+      (stroke (width 0.12) (type solid)) (layer "B.SilkS"))
+    (fp_arc (start 2.942335 1.078608) (mid 1.366487 1.987659) (end -0.29 1.235516)
+      (stroke (width 0.12) (type solid)) (layer "B.SilkS"))
+    (fp_line (start -1.15 -2.25) (end 3.7 -2.25)
+      (stroke (width 0.05) (type solid)) (layer "B.CrtYd"))
+    (fp_line (start -1.15 2.25) (end -1.15 -2.25)
+      (stroke (width 0.05) (type solid)) (layer "B.CrtYd"))
+    (fp_line (start 3.7 -2.25) (end 3.7 2.25)
+      (stroke (width 0.05) (type solid)) (layer "B.CrtYd"))
+    (fp_line (start 3.7 2.25) (end -1.15 2.25)
+      (stroke (width 0.05) (type solid)) (layer "B.CrtYd"))
+    (fp_line (start -0.23 1.16619) (end -0.23 -1.16619)
+      (stroke (width 0.1) (type solid)) (layer "B.Fab"))
+    (fp_arc (start -0.230555 -1.165476) (mid 3.17 -0.000452) (end -0.23 1.16619)
+      (stroke (width 0.1) (type solid)) (layer "B.Fab"))
+    (fp_circle (center 1.27 0) (end 2.77 0)
+      (stroke (width 0.1) (type solid)) (fill none) (layer "B.Fab"))
+    (pad "1" thru_hole rect (at 0 0 270) (size 1.8 1.8) (drill 0.9) (layers "*.Cu" "*.Mask")
+      (net 2 "GND") (pinfunction "K") (pintype "passive"))
+    (pad "2" thru_hole circle (at 2.54 0 270) (size 1.8 1.8) (drill 0.9) (layers "*.Cu" "*.Mask")
+      (net 29 "Net-(LED5-K)") (pinfunction "A") (pintype "passive"))
+    (model "${KICAD6_3DMODEL_DIR}/LED_THT.3dshapes/LED_D3.0mm.wrl"
+      (offset (xyz 0 0 0))
+      (scale (xyz 1 1 1))
+      (rotate (xyz 0 0 0))
+    )
+  )
   (footprint "Potentiometer_THT:Potentiometer redwiz" (layer "B.Cu")
     (at 163 113.31 180)
@@
   (segment (start 156.4 81.8) (end 159.83 81.8) (width 0.5) (layer "B.Cu") (net 1))
   (via (at 170.7 92.5) (size 0.8) (drill 0.4) (layers "F.Cu" "B.Cu") (free) (net 2))
-  (via (at 102.6 110.8) (size 0.8) (drill 0.4) (layers "F.Cu" "B.Cu") (free) (net 2))
   (via (at 115.5 100.7) (size 0.8) (drill 0.4) (layers "F.Cu" "B.Cu") (free) (net 2))
   (via (at 176.4 93.6) (size 0.8) (drill 0.4) (layers "F.Cu" "B.Cu") (free) (net 2))
@@
   (via (at 173.3 86.3) (size 0.8) (drill 0.4) (layers "F.Cu" "B.Cu") (free) (net 2))
   (via (at 168 75.6) (size 0.8) (drill 0.4) (layers "F.Cu" "B.Cu") (free) (net 2))
-  (via (at 93.6 110.8) (size 0.8) (drill 0.4) (layers "F.Cu" "B.Cu") (free) (net 2))
   (via (at 122 105) (size 0.8) (drill 0.4) (layers "F.Cu" "B.Cu") (free) (net 2))
   (via (at 114 78) (size 0.8) (drill 0.4) (layers "F.Cu" "B.Cu") (free) (net 2))
@@
   (segment (start 100.73 80.925) (end 100.73 84.3) (width 0.25) (layer "F.Cu") (net 28))
   (segment (start 91 101.7375) (end 91 107.7) (width 0.25) (layer "F.Cu") (net 29))
-  (segment (start 91.0125 107.7125) (end 100.4 107.7125) (width 0.25) (layer "F.Cu") (net 29))
-  (segment (start 91 107.7) (end 91.0125 107.7125) (width 0.25) (layer "F.Cu") (net 29))
+  (segment (start 100.2725 107.7125) (end 91.0125 107.7125) (width 0.25) (layer "F.Cu") (net 29))
+  (segment (start 91.0125 107.7125) (end 91 107.7) (width 0.25) (layer "F.Cu") (net 29))
+  (segment (start 100.74 108.18) (end 100.2725 107.7125) (width 0.25) (layer "F.Cu") (net 29))
+  (segment (start 102.04 109.475) (end 100.745 108.18) (width 0.25) (layer "F.Cu") (net 29))
+  (segment (start 100.745 108.18) (end 100.74 108.18) (width 0.25) (layer "F.Cu") (net 29))
   (segment (start 109.9 110.75) (end 114.25 110.75) (width 0.25) (layer "F.Cu") (net 30))
   (segment (start 123.7 113.7) (end 124.995 113.7) (width 0.25) (layer "F.Cu") (net 30))
