File: Punainen insinööri.kicad_sch (KiCad schematic)
At the start: 27 parts, among them J1 Barrel_Jack_Switch, Q1 MMBFJ113, SW1 SW_DPDT_x2, U1 LF351D

Commit message: jotain säätöä
Parts:
- added C9: 100uF, Capacitor_SMD:CP_Elec_6.3x5.4, symbol Device:C_Polarized_Small
- C8: footprint (none) -> Capacitor_SMD:CP_Elec_4x5.4
- J1: footprint (none) -> Connector_BarrelJack:BarrelJack_Horizontal
Connections:
- net +9V: now also C9.1
- net GND: now also C9.2
Other:
- moved on the sheet: C1
Changed lines of the file:
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@@
   (junction (at 115.57 38.1) (diameter 0) (color 0 0 0 0)
   )
+  (junction (at 52.07 50.8) (diameter 0) (color 0 0 0 0)
+  )
   (junction (at 99.06 57.15) (diameter 0) (color 0 0 0 0)
   )
@@
   (junction (at 106.68 41.91) (diameter 0) (color 0 0 0 0)
   )
-  (junction (at 77.47 49.53) (diameter 0) (color 0 0 0 0)
-  )
   (junction (at 148.59 58.42) (diameter 0) (color 0 0 0 0)
   )
@@
   (junction (at 90.17 76.2) (diameter 0) (color 0 0 0 0)
   )
+  (junction (at 52.07 55.88) (diameter 0) (color 0 0 0 0)
+  )
   (junction (at 99.06 76.2) (diameter 0) (color 0 0 0 0)
   )
@@
   (junction (at 106.68 38.1) (diameter 0) (color 0 0 0 0)
   )
-  (junction (at 77.47 76.2) (diameter 0) (color 0 0 0 0)
-  )
   (junction (at 148.59 38.1) (diameter 0) (color 0 0 0 0)
   )
@@
     (stroke (width 0) (type default))
   )
-  (wire (pts (xy 77.47 45.72) (xy 77.47 49.53))
-    (stroke (width 0) (type default))
-  )
-  (wire (pts (xy 71.12 67.31) (xy 86.36 67.31))
+  (wire (pts (xy 91.44 48.26) (xy 91.44 49.53))
+    (stroke (width 0) (type default))
+  )
+  (wire (pts (xy 85.09 67.31) (xy 86.36 67.31))
     (stroke (width 0) (type default))
   )
@@
     (stroke (width 0) (type default))
   )
-  (wire (pts (xy 77.47 76.2) (xy 77.47 77.47))
+  (wire (pts (xy 86.36 76.2) (xy 86.36 77.47))
     (stroke (width 0) (type default))
   )
@@
     (stroke (width 0) (type default))
   )
-  (wire (pts (xy 77.47 49.53) (xy 91.44 49.53))
-    (stroke (width 0) (type default))
-  )
   (wire (pts (xy 152.4 78.74) (xy 154.94 78.74))
     (stroke (width 0) (type default))
@@
     (stroke (width 0) (type default))
   )
-  (wire (pts (xy 77.47 49.53) (xy 77.47 60.96))
-    (stroke (width 0) (type default))
-  )
   (wire (pts (xy 99.06 76.2) (xy 106.68 76.2))
     (stroke (width 0) (type default))
@@
     (stroke (width 0) (type default))
   )
-  (wire (pts (xy 77.47 66.04) (xy 77.47 76.2))
-    (stroke (width 0) (type default))
-  )
   (wire (pts (xy 91.44 67.31) (xy 90.17 67.31))
     (stroke (width 0) (type default))
   )
+  (wire (pts (xy 57.15 55.88) (xy 52.07 55.88))
+    (stroke (width 0) (type default))
+  )
   (wire (pts (xy 193.04 54.61) (xy 189.23 54.61))
     (stroke (width 0) (type default))
   )
+  (wire (pts (xy 52.07 50.8) (xy 57.15 50.8))
+    (stroke (width 0) (type default))
+  )
   (wire (pts (xy 186.69 57.15) (xy 186.69 58.42))
     (stroke (width 0) (type default))
@@
     (stroke (width 0) (type default))
   )
-  (wire (pts (xy 77.47 76.2) (xy 86.36 76.2))
-    (stroke (width 0) (type default))
-  )
   (wire (pts (xy 106.68 41.91) (xy 106.68 62.23))
     (stroke (width 0) (type default))
@@
   )
   (wire (pts (xy 132.08 40.64) (xy 132.08 38.1))
+    (stroke (width 0) (type default))
+  )
+  (wire (pts (xy 41.91 50.8) (xy 52.07 50.8))
     (stroke (width 0) (type default))
   )
@@
     )
   )
-  (global_label "IN_red_pcb" (shape input) (at 71.12 67.31 180) (fields_autoplaced)
+  (global_label "IN_red_pcb" (shape input) (at 85.09 67.31 180) (fields_autoplaced)
     (effects (font (size 1.27 1.27)) (justify right))
-    (property "Intersheetrefs" "${INTERSHEET_REFS}" (at 57.9333 67.31 0)
+    (property "Intersheetrefs" "${INTERSHEET_REFS}" (at 71.9033 67.31 0)
       (effects (font (size 1.27 1.27)) (justify right) hide)
     )
@@
     )
   )
-  (symbol (lib_id "power:GND") (at 77.47 77.47 0) (unit 1)
-    (in_bom yes) (on_board yes) (dnp no)
-    (property "Reference" "#PWR02" (at 77.47 83.82 0)
-      (effects (font (size 1.27 1.27)) hide)
-    )
-    (property "Value" "GND" (at 77.47 81.28 0)
-      (effects (font (size 1.27 1.27)))
-    )
-    (property "Footprint" "" (at 77.47 77.47 0)
-      (effects (font (size 1.27 1.27)) hide)
-    )
-    (property "Datasheet" "" (at 77.47 77.47 0)
+  (symbol (lib_id "power:GND") (at 86.36 77.47 0) (unit 1)
+    (in_bom yes) (on_board yes) (dnp no)
+    (property "Reference" "#PWR02" (at 86.36 83.82 0)
+      (effects (font (size 1.27 1.27)) hide)
+    )
+    (property "Value" "GND" (at 86.36 81.28 0)
+      (effects (font (size 1.27 1.27)))
+    )
+    (property "Footprint" "" (at 86.36 77.47 0)
+      (effects (font (size 1.27 1.27)) hide)
+    )
+    (property "Datasheet" "" (at 86.36 77.47 0)
       (effects (font (size 1.27 1.27)) hide)
     )
@@
     )
   )
-  (symbol (lib_id "Device:C_Polarized_Small") (at 77.47 63.5 0) (unit 1)
+  (symbol (lib_id "Device:C_Polarized_Small") (at 57.15 53.34 0) (unit 1)
     (in_bom yes) (on_board yes) (dnp no) (fields_autoplaced)
-    (property "Reference" "C1" (at 80.01 62.3189 0)
-      (effects (font (size 1.27 1.27)) (justify left))
-    )
-    (property "Value" "100uF" (at 80.01 64.8589 0)
-      (effects (font (size 1.27 1.27)) (justify left))
-    )
-    (property "Footprint" "Capacitor_SMD:CP_Elec_6.3x5.4" (at 77.47 63.5 0)
-      (effects (font (size 1.27 1.27)) hide)
-    )
-    (property "Datasheet" "~" (at 77.47 63.5 0)
+    (property "Reference" "C1" (at 59.69 52.1589 0)
+      (effects (font (size 1.27 1.27)) (justify left))
+    )
+    (property "Value" "100uF" (at 59.69 54.6989 0)
+      (effects (font (size 1.27 1.27)) (justify left))
+    )
+    (property "Footprint" "Capacitor_SMD:CP_Elec_6.3x5.4" (at 57.15 53.34 0)
+      (effects (font (size 1.27 1.27)) hide)
+    )
+    (property "Datasheet" "~" (at 57.15 53.34 0)
       (effects (font (size 1.27 1.27)) hide)
     )
@@
       (effects (font (size 1.27 1.27)))
     )
-    (property "Footprint" "" (at 180.34 48.26 0)
+    (property "Footprint" "Capacitor_SMD:CP_Elec_4x5.4" (at 180.34 48.26 0)
       (effects (font (size 1.27 1.27)) hide)
     )
@@
     )
   )
-  (symbol (lib_id "power:+9V") (at 77.47 45.72 0) (unit 1)
+  (symbol (lib_id "Device:C_Polarized_Small") (at 52.07 53.34 0) (mirror y) (unit 1)
+    (in_bom yes) (on_board yes) (dnp no)
+    (property "Reference" "C9" (at 49.53 52.1589 0)
+      (effects (font (size 1.27 1.27)) (justify left))
+    )
+    (property "Value" "100uF" (at 49.53 54.6989 0)
+      (effects (font (size 1.27 1.27)) (justify left))
+    )
+    (property "Footprint" "Capacitor_SMD:CP_Elec_6.3x5.4" (at 52.07 53.34 0)
+      (effects (font (size 1.27 1.27)) hide)
+    )
+    (property "Datasheet" "~" (at 52.07 53.34 0)
+      (effects (font (size 1.27 1.27)) hide)
+    )
+    (pin "1")
+    (pin "2")
+    (instances
+      (project "Punainen insinööri"
+        (path "/e5ef43d6-cafc-424f-9222-4ed75d8d1dc6"
+          (reference "C9") (unit 1)
+        )
+      )
+    )
+  )
+  (symbol (lib_id "power:+9V") (at 91.44 48.26 0) (unit 1)
     (in_bom yes) (on_board yes) (dnp no) (fields_autoplaced)
-    (property "Reference" "#PWR01" (at 77.47 49.53 0)
-      (effects (font (size 1.27 1.27)) hide)
-    )
-    (property "Value" "+9V" (at 77.47 41.91 0)
-      (effects (font (size 1.27 1.27)))
-    )
-    (property "Footprint" "" (at 77.47 45.72 0)
-      (effects (font (size 1.27 1.27)) hide)
-    )
-    (property "Datasheet" "" (at 77.47 45.72 0)
+    (property "Reference" "#PWR01" (at 91.44 52.07 0)
+      (effects (font (size 1.27 1.27)) hide)
+    )
+    (property "Value" "+9V" (at 91.44 44.45 0)
+      (effects (font (size 1.27 1.27)))
+    )
+    (property "Footprint" "" (at 91.44 48.26 0)
+      (effects (font (size 1.27 1.27)) hide)
+    )
+    (property "Datasheet" "" (at 91.44 48.26 0)
       (effects (font (size 1.27 1.27)) hide)
     )
@@
     )
   )
+  (symbol (lib_id "power:GND") (at 52.07 55.88 0) (unit 1)
+    (in_bom yes) (on_board yes) (dnp no)
+    (property "Reference" "#PWR05" (at 52.07 62.23 0)
+      (effects (font (size 1.27 1.27)) hide)
+    )
+    (property "Value" "GND" (at 52.07 59.69 0)
+      (effects (font (size 1.27 1.27)))
+    )
+    (property "Footprint" "" (at 52.07 55.88 0)
+      (effects (font (size 1.27 1.27)) hide)
+    )
+    (property "Datasheet" "" (at 52.07 55.88 0)
+      (effects (font (size 1.27 1.27)) hide)
+    )
+    (pin "1")
+    (instances
+      (project "Punainen insinööri"
+        (path "/e5ef43d6-cafc-424f-9222-4ed75d8d1dc6"
+          (reference "#PWR05") (unit 1)
+        )
+      )
+    )
+  )
   (symbol (lib_id "Device:C_Small") (at 153.67 38.1 270) (unit 1)
     (in_bom yes) (on_board yes) (dnp no)
@@
       (effects (font (size 1.27 1.27)) hide)
     )
-    (property "Footprint" "" (at 25.4 52.324 0)
-      (effects (font (size 1.27 1.27)) hide)
-    )
+    (property "Footprint" "Connector_BarrelJack:BarrelJack_Horizontal" (at 25.4 52.324 0)
+      (effects (font (size 1.27 1.27)) hide)
+    )

Commit message: the trans question
Parts:
- Q1: value MMBFJ113 -> MMBF4393LT1G; LCSC # (none) -> C152291
Connections:
- no-connect marks 0 -> 2
Changed lines of the file:
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@@
   (junction (at 111.76 38.1) (diameter 0) (color 0 0 0 0)
   )
+  (no_connect (at 120.65 67.31))
+  (no_connect (at 118.11 67.31))
   (wire (pts (xy 86.36 67.31) (xy 86.36 69.85))
     (stroke (width 0) (type default))
@@
       (effects (font (size 1.27 1.27)) (justify left))
     )
-    (property "Value" "MMBFJ113" (at 171.45 40.005 0)
+    (property "Value" "MMBF4393LT1G" (at 171.45 40.005 0)
       (effects (font (size 1.27 1.27)) (justify left))
     )
@@
       (effects (font (size 1.27 1.27)) (justify left) hide)
     )
-    (pin "1")
+    (property "LCSC #" "C152291" (at 166.37 38.1 0)
+      (effects (font (size 1.27 1.27)) hide)
+    )
+    (pin "1")

Commit message: small fixes
Parts:
- added C10: 10nF, Capacitor_SMD:C_0805_2012Metric_Pad1.18x1.45mm_HandSolder, symbol Device:C_Small
- added D2, D3: 1N4148W, Diode_SMD:D_SOD-123, symbol Diode:1N4148W
- added LED3, LED4: LED_Small, symbol Device:LED_Small
- added Q2, Q3: MMBF170, Package_TO_SOT_SMD:SOT-23, symbol Transistor_FET:MMBF170
- added R10, R11: 4.7k, Resistor_SMD:R_0805_2012Metric_Pad1.20x1.40mm_HandSolder, symbol Device:R_Small
Connections:
- net +9V: now also C10.1, D2.1 (K), D3.1 (K), Q2.3 (D), Q3.3 (D)
- net FS_red: now also D2.2 (A), Q2.1 (G)
- net GND: now also C10.2, LED3.1 (K), LED4.1 (K)
- new net: LED3.2 (A), R10.2
- new net: LED4.2 (A), R11.2
- new net: Q3.2 (S), R11.1
- new net: Q2.2 (S), R10.1
- new net FS_engi: D3.2 (A), Q3.1 (G)
Other:
- note added: "engi bypass"
- note added: "power"
- note added: "red bypass"
- moved on the sheet: C2, C3, C4, C5, C6, C7, C8, Q1, R1, R2, R3, R4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

Commit message: millenials in shambles
Parts:
- LED1, LED2: footprint (none) -> LED_SMD:LED_1206_3216Metric_Pad1.42x1.75mm_HandSolder
Changed lines of the file:
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@@
       (effects (font (size 1.27 1.27)) hide)
     )
-    (property "Footprint" "" (at 59.69 36.83 90)
-      (effects (font (size 1.27 1.27)) hide)
-    )
-    (property "Datasheet" "~" (at 59.69 36.83 90)
+    (property "Footprint" "LED_SMD:LED_1206_3216Metric_Pad1.42x1.75mm_HandSolder" (at 59.69 36.83 90)
+      (effects (font (size 1.27 1.27)) hide)
+    )
+    (property "Datasheet" "C2827254" (at 59.69 36.83 90)
       (effects (font (size 1.27 1.27)) hide)
     )
@@
       (effects (font (size 1.27 1.27)) hide)
     )
-    (property "Footprint" "" (at 59.69 40.64 90)
-      (effects (font (size 1.27 1.27)) hide)
-    )
-    (property "Datasheet" "~" (at 59.69 40.64 90)
-      (effects (font (size 1.27 1.27)) hide)
-    )
+    (property "Footprint" "LED_SMD:LED_1206_3216Metric_Pad1.42x1.75mm_HandSolder" (at 59.69 40.64 90)
+      (effects (font (size 1.27 1.27)) hide)
+    )
+    (property "Datasheet" "C2827254" (at 59.69 40.64 90)
+      (effects (font (size 1.27 1.27)) hide)
+    )

Commit message: Schema valmiina
Parts:
- added C11, C12, C14: 10nF, Capacitor_SMD:C_0805_2012Metric_Pad1.18x1.45mm_HandSolder, symbol Device:C_Small
- added C13, C18, C19: 1uF, Capacitor_SMD:C_0805_2012Metric_Pad1.18x1.45mm_HandSolder, symbol Device:C_Small
- added C15: 100pF, Capacitor_SMD:C_0805_2012Metric_Pad1.18x1.45mm_HandSolder, symbol Device:C_Small
- added C16: 4.7nF, Capacitor_SMD:C_0805_2012Metric_Pad1.18x1.45mm_HandSolder, symbol Device:C_Small
- added C17: 10uF, Capacitor_SMD:CP_Elec_4x5.4, symbol Device:C_Polarized_Small
- added D4, D5, D6: 1N4148W, Diode_SMD:D_SOD-123, symbol Diode:1N4148W
- added LED5, LED6: LED_Small, LED_SMD:LED_1206_3216Metric_Pad1.42x1.75mm_HandSolder, symbol Device:LED_Small
- added Q4: BC807, Package_TO_SOT_SMD:SOT-23, symbol Transistor_BJT:BC807
- added R12, R13, R19, R20, R21: 10k, Resistor_SMD:R_0805_2012Metric_Pad1.20x1.40mm_HandSolder, symbol Device:R_Small
- added R14, R15, R16, R18, R27: 1M, Resistor_SMD:R_0805_2012Metric_Pad1.20x1.40mm_HandSolder, symbol Device:R_Small
- added R17, R23, R26, R28: 1k, Resistor_SMD:R_0805_2012Metric_Pad1.20x1.40mm_HandSolder, symbol Device:R_Small
- added R22: 220Ω, Resistor_SMD:R_0805_2012Metric_Pad1.20x1.40mm_HandSolder, symbol Device:R_Small
- added R24: 470k, Resistor_SMD:R_0805_2012Metric_Pad1.20x1.40mm_HandSolder, symbol Device:R_Small
- added R25: 100Ω, Resistor_SMD:R_1206_3216Metric_Pad1.30x1.75mm_HandSolder, symbol Device:R_Small
- added SW2: SW_DPDT_x2, Button_Switch_THT:SW_Push_2P2T_Toggle_CK_PVA2xxH1xxxxxxV2, symbol Switch:SW_DPDT_x2
- added U2: TL074, Package_SO:SO-14_3.9x8.65mm_P1.27mm, symbol Amplifier_Operational:TL074
- added U3: LM13700, Package_SO:SOP-16_3.9x9.9mm_P1.27mm, symbol Amplifier_Operational:LM13700
- added rv4: 1M, symbol Device:R_Potentiometer_Small
- added rv5: 10k, symbol Device:R_Potentiometer_Small
- added rv6: 100k, symbol Device:R_Potentiometer_Small
- rv1: renamed from int1; value 1M log -> 1M; Kenttä4 (none) -> Intesity log
- rv2: renamed from tone1; value 100k lin -> 100k; Kenttä4 (none) -> tone linear
- rv3: renamed from volume1; value 100k log -> 100k; Kenttä4 (none) -> volume log
Connections:
- net +9V: now also C11.1, C12.1, R12.1, R14.1, U2.4 (V+), U3.11 (V+)
- net FS_engi: now also SW2.6 (C)
- net GND: now also C11.2, C12.2, C13.1, C18.2, C19.2, LED5.2 (A), LED6.1 (K), R13.2, R15.2, R16.2, U2.11 (V-), U3.16, U3.6 (V-), rv5.3
- net IN_red: now reaches SW1.2 (B)
- net IN_red: now also SW2.3 (C), SW2.4 (A)
- net OUT_red: now reaches SW1.3 (C), SW1.4 (A)
- new net: D6.2 (A), Q4.1 (B), U2.14
- new net: D6.1 (K), Q4.2 (E), R28.2, U2.13 (-)
- new net: Q4.3 (C), R27.2, U3.1
- new net: C18.1, R24.1, R26.1, rv6.2, rv6.3
- new net: D4.1 (K), R24.2, U2.6 (-)
- new net: C14.1, R18.2, U2.10 (+), U2.5 (+)
- new net: C14.2, LED5.1 (K), LED6.2 (A), R17.2
- new net: U3.7, U3.8
- new net: D4.2 (A), D5.1 (K), U2.7
- new net: D5.2 (A), R25.1
- new net: R25.2, rv6.1
- new net: C16.1, R19.1
- new net: C15.2, R19.2, R20.2, U2.9 (-), U3.5, rv4.2
- new net: C13.2, R14.2, R15.1, U2.3 (+)
- new net: R21.1, R22.2, U3.3 (+)
- new net: C19.1, R26.2, U2.12 (+)
- new net: R12.2, R13.1, U3.14 (+)
- new net: U3.12, U3.13 (-)
- new net: C15.1, R21.2, R23.1, U2.8, rv4.1
- new net: U3.10, U3.9
- new net: C17.1, R23.2
- new net: C17.2, rv5.1
- new net +5V: C16.2, R18.1, R20.1, R22.1, R27.1, R28.1, U2.1, U2.2 (-), U3.4 (-)
- new net IN_engi: SW2.2 (B)
- new net IN_engi_pcb: R16.1, R17.1, SW2.1 (A)
- new net OUT_engi_pcb: SW2.5 (B), rv5.2
- no-connect marks 2 -> 5
Other:
- note added: "Engineer's thumb"
- note added: "Op amp bdsm"
- note added: "Red Fuzz"
- note added: "engi switch"
- note added: "red switch"
- moved on the sheet: C1, C10, C2, C3, C4, C5, C6, C7, C8, C9, D1, D2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

Commit message: pieniä muutoksia
Parts:
- SW1: footprint (none) -> Button_Switch_THT:SW_Push_2P2T_Toggle_CK_PVA2xxH1xxxxxxV2
- rv1, rv2, rv3, rv4, rv5, rv6: footprint (none) -> Potentiometer_THT:Potentiometer redwiz
Changed lines of the file:
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@@
       (effects (font (size 1.27 1.27)))
     )
-    (property "Footprint" "" (at 256.54 22.86 0)
+    (property "Footprint" "Button_Switch_THT:SW_Push_2P2T_Toggle_CK_PVA2xxH1xxxxxxV2" (at 256.54 22.86 0)
       (effects (font (size 1.27 1.27)) hide)
     )
@@
       (effects (font (size 1.27 1.27)))
     )
-    (property "Footprint" "" (at 62.23 24.13 0)
+    (property "Footprint" "Potentiometer_THT:Potentiometer redwiz" (at 62.23 24.13 0)
       (effects (font (size 1.27 1.27)) hide)
     )
@@
       (effects (font (size 1.27 1.27)))
     )
-    (property "Footprint" "" (at 140.97 57.15 0)
+    (property "Footprint" "Potentiometer_THT:Potentiometer redwiz" (at 140.97 57.15 0)
       (effects (font (size 1.27 1.27)) hide)
     )
@@
       (effects (font (size 1.27 1.27)))
     )
-    (property "Footprint" "" (at 87.63 120.65 0)
+    (property "Footprint" "Potentiometer_THT:Potentiometer redwiz" (at 87.63 120.65 0)
       (effects (font (size 1.27 1.27)) hide)
     )
@@
       (effects (font (size 1.27 1.27)))
     )
-    (property "Footprint" "" (at 90.17 95.25 0)
+    (property "Footprint" "Potentiometer_THT:Potentiometer redwiz" (at 90.17 95.25 0)
       (effects (font (size 1.27 1.27)) hide)
     )
@@
       (effects (font (size 1.27 1.27)))
     )
-    (property "Footprint" "" (at 90.17 44.45 0)
+    (property "Footprint" "Potentiometer_THT:Potentiometer redwiz" (at 90.17 44.45 0)
       (effects (font (size 1.27 1.27)) hide)
     )
@@
       (effects (font (size 1.27 1.27)))
     )
-    (property "Footprint" "" (at 139.7 105.41 0)
+    (property "Footprint" "Potentiometer_THT:Potentiometer redwiz" (at 139.7 105.41 0)
       (effects (font (size 1.27 1.27)) hide)
     )
@@
       (effects (font (size 1.27 1.27)))
     )
-    (property "Footprint" "" (at 256.54 36.83 0)
-      (effects (font (size 1.27 1.27)) hide)
-    )
+    (property "Footprint" "Button_Switch_THT:SW_Push_2P2T_Toggle_CK_PVA2xxH1xxxxxxV2" (at 256.54 36.83 0)
+      (effects (font (size 1.27 1.27)) hide)
+    )

Commit message: pcb v1
Parts:
- C1, C9: LCSC# (none) -> C37308
- C10, C11, C12, C14: LCSC# (none) -> C58456
- C13, C18, C19: LCSC# (none) -> C520051
- C15: LCSC# (none) -> C525281
- C16: LCSC# (none) -> C376986
- C17, C8: LCSC# (none) -> C4747969
- C2: LCSC# (none) -> C520039
- C3: LCSC# (none) -> C376859
- C4: LCSC# (none) -> C541526
- C5, C7: LCSC# (none) -> C282730
- C6: LCSC# (none) -> C1322372
- D1: LCSC# (none) -> C2892326
- D2, D3, D4, D5, D6: LCSC# (none) -> C5345962
- J1: LCSC# (none) -> C194407; now left out of the parts list
- LED1, LED2, LED5, LED6: LCSC# (none) -> C84263
- LED3, LED4, SW1, SW2, rv1, rv2, rv3, rv4, rv5, rv6: now left out of the parts list
- Q1: LCSC # C152291 -> (none); LCSC# (none) -> C152291
- Q2, Q3: LCSC# (none) -> C5330373
- Q4: LCSC# (none) -> C5184433
- R1, R2, R24: LCSC# (none) -> C2960743
- R10, R11: LCSC# (none) -> C2907264
- R12, R13, R19, R20, R21, R5, R8: LCSC# (none) -> C17414
- R14, R15, R16, R18, R27, R3, R7: LCSC# (none) -> C103906
- R17, R23, R26, R28: LCSC# (none) -> C2907232
- R22: LCSC# (none) -> C2933369
- R25: LCSC# (none) -> C3016626
- R4: LCSC# (none) -> C17398
- R6: LCSC# (none) -> C104106
- R9: LCSC# (none) -> C153384
- U1: LCSC# (none) -> C1346659
- U2: LCSC# (none) -> C107644
- U3: LCSC# (none) -> C5160094
