File: Punainen insinööri.kicad_sch (KiCad schematic)
At the start: 75 parts, among them J1 Barrel_Jack_Switch, Q1 MMBF4393LT1G, Q2 MMBF170, Q3 MMBF170, Q4 BC807, SW1 SW_DPDT_x2, SW2 SW_DPDT_x2, U1 LF351D, U2 TL074, U3 LM13700

Commit message: Konkan tuplaus temppu
Parts:
- added C20, C21: 10uF, Capacitor_SMD:CP_Elec_4x5.4, symbol Device:C_Polarized_Small
- added C22, C23: 100uF, Capacitor_SMD:CP_Elec_6.3x5.4, symbol Device:C_Polarized_Small
Connections:
- net +9V: now also C22.1, C23.1
- net GND: now also C22.2, C23.2
- net at C8.1, Q1.2 (S), R8.1: now also C21.1
- net at C8.2, rv3.3: now also C21.2
- net at C17.1, R23.2: now also C20.1
- net at C17.2, rv5.1: now also C20.2
Changed lines of the file:
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@@
   (junction (at 127 90.17) (diameter 0) (color 0 0 0 0)
   )
+  (junction (at 194.31 121.92) (diameter 0) (color 0 0 0 0)
+  )
   (junction (at 270.51 109.22) (diameter 0) (color 0 0 0 0)
   )
+  (junction (at 140.97 50.8) (diameter 0) (color 0 0 0 0)
+  )
   (junction (at 33.02 52.07) (diameter 0) (color 0 0 0 0)
   )
@@
   (junction (at 53.34 31.75) (diameter 0) (color 0 0 0 0)
   )
+  (junction (at 129.54 50.8) (diameter 0) (color 0 0 0 0)
+  )
   (junction (at 102.87 60.96) (diameter 0) (color 0 0 0 0)
   )
@@
   (junction (at 62.23 113.03) (diameter 0) (color 0 0 0 0)
   )
+  (junction (at 134.62 90.17) (diameter 0) (color 0 0 0 0)
+  )
   (junction (at 45.72 60.96) (diameter 0) (color 0 0 0 0)
   )
   (junction (at 64.77 27.94) (diameter 0) (color 0 0 0 0)
   )
+  (junction (at 194.31 116.84) (diameter 0) (color 0 0 0 0)
+  )
   (junction (at 68.58 130.81) (diameter 0) (color 0 0 0 0)
   )
@@
   (junction (at 86.36 44.45) (diameter 0) (color 0 0 0 0)
   )
+  (junction (at 139.7 97.79) (diameter 0) (color 0 0 0 0)
+  )
   (junction (at 80.01 130.81) (diameter 0) (color 0 0 0 0)
   )
@@
     (stroke (width 0) (type default))
   )
+  (wire (pts (xy 191.77 116.84) (xy 194.31 116.84))
+    (stroke (width 0) (type default))
+  )
   (wire (pts (xy 241.3 146.05) (xy 241.3 147.32))
     (stroke (width 0) (type default))
@@
     (stroke (width 0) (type default))
   )
+  (wire (pts (xy 191.77 121.92) (xy 194.31 121.92))
+    (stroke (width 0) (type default))
+  )
   (wire (pts (xy 96.52 130.81) (xy 88.9 130.81))
     (stroke (width 0) (type default))
@@
     (stroke (width 0) (type default))
   )
+  (wire (pts (xy 137.16 43.18) (xy 140.97 43.18))
+    (stroke (width 0) (type default))
+  )
+  (wire (pts (xy 134.62 90.17) (xy 134.62 97.79))
+    (stroke (width 0) (type default))
+  )
   (wire (pts (xy 207.01 58.42) (xy 209.55 58.42))
     (stroke (width 0) (type default))
@@
     (stroke (width 0) (type default))
   )
+  (wire (pts (xy 139.7 97.79) (xy 139.7 102.87))
+    (stroke (width 0) (type default))
+  )
   (wire (pts (xy 248.92 125.73) (xy 259.08 125.73))
     (stroke (width 0) (type default))
@@
     (stroke (width 0) (type default))
   )
+  (wire (pts (xy 129.54 43.18) (xy 129.54 50.8))
+    (stroke (width 0) (type default))
+  )
   (wire (pts (xy 247.65 125.73) (xy 247.65 124.46))
     (stroke (width 0) (type default))
@@
     (stroke (width 0) (type default))
   )
+  (wire (pts (xy 194.31 116.84) (xy 196.85 116.84))
+    (stroke (width 0) (type default))
+  )
   (wire (pts (xy 74.93 99.06) (xy 64.77 99.06))
     (stroke (width 0) (type default))
@@
     (stroke (width 0) (type default))
   )
-  (wire (pts (xy 123.19 50.8) (xy 132.08 50.8))
+  (wire (pts (xy 123.19 50.8) (xy 129.54 50.8))
     (stroke (width 0) (type default))
   )
@@
     (stroke (width 0) (type default))
   )
-  (wire (pts (xy 139.7 90.17) (xy 139.7 102.87))
+  (wire (pts (xy 139.7 90.17) (xy 139.7 97.79))
     (stroke (width 0) (type default))
   )
@@
     (stroke (width 0) (type default))
   )
+  (wire (pts (xy 194.31 121.92) (xy 196.85 121.92))
+    (stroke (width 0) (type default))
+  )
   (wire (pts (xy 127 91.44) (xy 127 90.17))
     (stroke (width 0) (type default))
@@
     (stroke (width 0) (type default))
   )
+  (wire (pts (xy 140.97 43.18) (xy 140.97 50.8))
+    (stroke (width 0) (type default))
+  )
   (wire (pts (xy 78.74 27.94) (xy 64.77 27.94))
     (stroke (width 0) (type default))
@@
     (stroke (width 0) (type default))
   )
+  (wire (pts (xy 129.54 50.8) (xy 132.08 50.8))
+    (stroke (width 0) (type default))
+  )
   (wire (pts (xy 104.14 96.52) (xy 102.87 96.52))
     (stroke (width 0) (type default))
@@
     (stroke (width 0) (type default))
   )
+  (wire (pts (xy 132.08 43.18) (xy 129.54 43.18))
+    (stroke (width 0) (type default))
+  )
   (wire (pts (xy 82.55 120.65) (xy 85.09 120.65))
     (stroke (width 0) (type default))
@@
   (symbol (lib_id "Transistor_FET:MMBFJ113") (at 120.65 44.45 0) (unit 1)
     (in_bom yes) (on_board yes) (dnp no)
-    (property "Reference" "Q1" (at 124.46 40.64 0)
+    (property "Reference" "Q1" (at 118.11 38.1 0)
       (effects (font (size 1.27 1.27)) (justify left))
     )
-    (property "Value" "MMBF4393LT1G" (at 124.46 43.18 0)
+    (property "Value" "MMBF4393LT1G" (at 106.68 35.56 0)
       (effects (font (size 1.27 1.27)) (justify left))
     )
@@
     )
   )
+  (symbol (lib_id "Device:C_Polarized_Small") (at 191.77 119.38 0) (mirror y) (unit 1)
+    (in_bom yes) (on_board yes) (dnp no)
+    (property "Reference" "C22" (at 189.23 118.1989 0)
+      (effects (font (size 1.27 1.27)) (justify left))
+    )
+    (property "Value" "100uF" (at 189.23 120.7389 0)
+      (effects (font (size 1.27 1.27)) (justify left))
+    )
+    (property "Footprint" "Capacitor_SMD:CP_Elec_6.3x5.4" (at 191.77 119.38 0)
+      (effects (font (size 1.27 1.27)) hide)
+    )
+    (property "Datasheet" "~" (at 191.77 119.38 0)
+      (effects (font (size 1.27 1.27)) hide)
+    )
+    (property "LCSC#" "C37308" (at 191.77 119.38 0)
+      (effects (font (size 1.27 1.27)) hide)
+    )
+    (pin "1")
+    (pin "2")
+    (instances
+      (project "Punainen insinööri"
+        (path "/e5ef43d6-cafc-424f-9222-4ed75d8d1dc6"
+          (reference "C22") (unit 1)
+        )
+      )
+    )
+  )
   (symbol (lib_id "Device:R_Small") (at 55.88 24.13 270) (mirror x) (unit 1)
     (in_bom yes) (on_board yes) (dnp no)
@@
     )
   )
+  (symbol (lib_id "Device:C_Polarized_Small") (at 196.85 119.38 0) (unit 1)
+    (in_bom yes) (on_board yes) (dnp no) (fields_autoplaced)
+    (property "Reference" "C23" (at 199.39 118.1989 0)
+      (effects (font (size 1.27 1.27)) (justify left))
+    )
+    (property "Value" "100uF" (at 199.39 120.7389 0)
+      (effects (font (size 1.27 1.27)) (justify left))
+    )
+    (property "Footprint" "Capacitor_SMD:CP_Elec_6.3x5.4" (at 196.85 119.38 0)
+      (effects (font (size 1.27 1.27)) hide)
+    )
+    (property "Datasheet" "~" (at 196.85 119.38 0)
+      (effects (font (size 1.27 1.27)) hide)
+    )
+    (property "LCSC#" "C37308" (at 196.85 119.38 0)
+      (effects (font (size 1.27 1.27)) hide)
+    )
+    (pin "1")
+    (pin "2")
+    (instances
+      (project "Punainen insinööri"
+        (path "/e5ef43d6-cafc-424f-9222-4ed75d8d1dc6"
+          (reference "C23") (unit 1)
+        )
+      )
+    )
+  )
+  (symbol (lib_id "Device:C_Polarized_Small") (at 137.16 97.79 90) (unit 1)
+    (in_bom yes) (on_board yes) (dnp no) (fields_autoplaced)
+    (property "Reference" "C20" (at 136.6139 92.71 90)
+      (effects (font (size 1.27 1.27)))
+    )
+    (property "Value" "10uF" (at 136.6139 95.25 90)
+      (effects (font (size 1.27 1.27)))
+    )
+    (property "Footprint" "Capacitor_SMD:CP_Elec_4x5.4" (at 137.16 97.79 0)
+      (effects (font (size 1.27 1.27)) hide)
+    )
+    (property "Datasheet" "~" (at 137.16 97.79 0)
+      (effects (font (size 1.27 1.27)) hide)
+    )
+    (property "LCSC#" "C4747969" (at 137.16 97.79 0)
+      (effects (font (size 1.27 1.27)) hide)
+    )
+    (pin "1")
+    (pin "2")
+    (instances
+      (project "Punainen insinööri"
+        (path "/e5ef43d6-cafc-424f-9222-4ed75d8d1dc6"
+          (reference "C20") (unit 1)
+        )
+      )
+    )
+  )
   (symbol (lib_id "power:GND") (at 207.01 35.56 0) (unit 1)
     (in_bom yes) (on_board yes) (dnp no)
@@
     )
   )
+  (symbol (lib_id "power:+9V") (at 194.31 116.84 0) (unit 1)
+    (in_bom yes) (on_board yes) (dnp no) (fields_autoplaced)
+    (property "Reference" "#PWR022" (at 194.31 120.65 0)
+      (effects (font (size 1.27 1.27)) hide)
+    )
+    (property "Value" "+9V" (at 194.31 113.03 0)
+      (effects (font (size 1.27 1.27)))
+    )
+    (property "Footprint" "" (at 194.31 116.84 0)
+      (effects (font (size 1.27 1.27)) hide)
+    )
+    (property "Datasheet" "" (at 194.31 116.84 0)
+      (effects (font (size 1.27 1.27)) hide)
+    )
+    (pin "1")
+    (instances
+      (project "Punainen insinööri"
+        (path "/e5ef43d6-cafc-424f-9222-4ed75d8d1dc6"
+          (reference "#PWR022") (unit 1)
+        )
+      )
+    )
+  )
   (symbol (lib_id "power:GND") (at 228.6 88.9 0) (unit 1)
     (in_bom yes) (on_board yes) (dnp no)
@@
     )
   )
+  (symbol (lib_id "Device:C_Polarized_Small") (at 134.62 43.18 90) (unit 1)
+    (in_bom yes) (on_board yes) (dnp no) (fields_autoplaced)
+    (property "Reference" "C21" (at 134.0739 38.1 90)
+      (effects (font (size 1.27 1.27)))
+    )
+    (property "Value" "10uF" (at 134.0739 40.64 90)
+      (effects (font (size 1.27 1.27)))
+    )
+    (property "Footprint" "Capacitor_SMD:CP_Elec_4x5.4" (at 134.62 43.18 0)
+      (effects (font (size 1.27 1.27)) hide)
+    )
+    (property "Datasheet" "~" (at 134.62 43.18 0)
+      (effects (font (size 1.27 1.27)) hide)
+    )
+    (property "LCSC#" "C4747969" (at 134.62 43.18 0)
+      (effects (font (size 1.27 1.27)) hide)
+    )
+    (pin "1")
+    (pin "2")
+    (instances
+      (project "Punainen insinööri"
+        (path "/e5ef43d6-cafc-424f-9222-4ed75d8d1dc6"
+          (reference "C21") (unit 1)
+        )
+      )
+    )
+  )
   (symbol (lib_id "Device:R_Small") (at 130.81 90.17 90) (mirror x) (unit 1)
     (in_bom yes) (on_board yes) (dnp no)
@@
         )
       )
+    )
+  )
+  (symbol (lib_id "power:GND") (at 194.31 121.92 0) (unit 1)
+    (in_bom yes) (on_board yes) (dnp no)
+    (property "Reference" "#PWR023" (at 194.31 128.27 0)
+      (effects (font (size 1.27 1.27)) hide)
+    )
+    (property "Value" "GND" (at 194.31 125.73 0)
+      (effects (font (size 1.27 1.27)))
+    )
+    (property "Footprint" "" (at 194.31 121.92 0)
+      (effects (font (size 1.27 1.27)) hide)
+    )
+    (property "Datasheet" "" (at 194.31 121.92 0)
+      (effects (font (size 1.27 1.27)) hide)
+    )
+    (pin "1")
+    (instances
+      (project "Punainen insinööri"
+        (path "/e5ef43d6-cafc-424f-9222-4ed75d8d1dc6"
+          (reference "#PWR023") (unit 1)
+        )
+      )
