File: Punainen insinööri.kicad_sch (KiCad schematic)
At the start: 79 parts, among them J1 Barrel_Jack_Switch, Q1 MMBF4393LT1G, Q2 MMBF170, Q3 MMBF170, Q4 BC807, SW1 SW_DPDT_x2, SW2 SW_DPDT_x2, U1 LF351D, U2 TL074, U3 LM13700

Commit message: Ledin lisäys loitsu
Parts:
- added LED7, LED8: LED_Small, LED_THT:LED_D3.0mm, symbol Device:LED_Small
Connections:
- net GND: now also LED7.1 (K), LED8.1 (K)
- net at C14.2, LED5.1 (K), LED6.2 (A)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: now also LED7.2 (A), LED8.2 (A)
Changed lines of the file:
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@@
   (junction (at 119.38 113.03) (diameter 0) (color 0 0 0 0)
   )
+  (junction (at 39.37 133.35) (diameter 0) (color 0 0 0 0)
+  )
   (junction (at 127 96.52) (diameter 0) (color 0 0 0 0)
   )
@@
   (junction (at 123.19 60.96) (diameter 0) (color 0 0 0 0)
   )
+  (junction (at 41.91 133.35) (diameter 0) (color 0 0 0 0)
+  )
   (junction (at 113.03 60.96) (diameter 0) (color 0 0 0 0)
   )
@@
   (junction (at 40.64 118.11) (diameter 0) (color 0 0 0 0)
   )
+  (junction (at 45.72 139.7) (diameter 0) (color 0 0 0 0)
+  )
   (junction (at 207.01 29.21) (diameter 0) (color 0 0 0 0)
   )
@@
   (junction (at 78.74 44.45) (diameter 0) (color 0 0 0 0)
   )
+  (junction (at 35.56 139.7) (diameter 0) (color 0 0 0 0)
+  )
   (junction (at 45.72 52.07) (diameter 0) (color 0 0 0 0)
   )
@@
     (stroke (width 0) (type default))
   )
+  (wire (pts (xy 39.37 133.35) (xy 40.64 133.35))
+    (stroke (width 0) (type default))
+  )
   (wire (pts (xy 127 97.79) (xy 127 96.52))
     (stroke (width 0) (type default))
@@
     (stroke (width 0) (type default))
   )
-  (wire (pts (xy 41.91 139.7) (xy 80.01 139.7))
+  (wire (pts (xy 35.56 139.7) (xy 39.37 139.7))
+    (stroke (width 0) (type default))
+  )
+  (wire (pts (xy 41.91 139.7) (xy 45.72 139.7))
     (stroke (width 0) (type default))
   )
@@
     (stroke (width 0) (type default))
   )
-  (wire (pts (xy 39.37 133.35) (xy 40.64 133.35))
+  (wire (pts (xy 35.56 133.35) (xy 39.37 133.35))
     (stroke (width 0) (type default))
   )
@@
     (stroke (width 0) (type default))
   )
+  (wire (pts (xy 41.91 133.35) (xy 45.72 133.35))
+    (stroke (width 0) (type default))
+  )
   (wire (pts (xy 45.72 52.07) (xy 45.72 54.61))
     (stroke (width 0) (type default))
@@
     (stroke (width 0) (type default))
   )
-  (wire (pts (xy 31.75 139.7) (xy 39.37 139.7))
+  (wire (pts (xy 31.75 139.7) (xy 35.56 139.7))
     (stroke (width 0) (type default))
   )
@@
     (stroke (width 0) (type default))
   )
+  (wire (pts (xy 35.56 134.62) (xy 35.56 133.35))
+    (stroke (width 0) (type default))
+  )
   (wire (pts (xy 270.51 137.16) (xy 267.97 137.16))
     (stroke (width 0) (type default))
@@
     (stroke (width 0) (type default))
   )
+  (wire (pts (xy 45.72 133.35) (xy 45.72 134.62))
+    (stroke (width 0) (type default))
+  )
   (wire (pts (xy 31.75 118.11) (xy 30.48 118.11))
     (stroke (width 0) (type default))
@@
     (stroke (width 0) (type default))
   )
+  (wire (pts (xy 45.72 139.7) (xy 80.01 139.7))
+    (stroke (width 0) (type default))
+  )
   (rectangle (start 233.68 102.87) (end 281.94 161.29)
     (stroke (width 0) (type default))
@@
     )
   )
+  (symbol (lib_id "Device:LED_Small") (at 35.56 137.16 270) (mirror x) (unit 1)
+    (in_bom yes) (on_board yes) (dnp no)
+    (property "Reference" "LED8" (at 38.1 137.16 0)
+      (effects (font (size 1.27 1.27)) hide)
+    )
+    (property "Value" "LED_Small" (at 38.1 137.0965 0)
+      (effects (font (size 1.27 1.27)) hide)
+    )
+    (property "Footprint" "LED_THT:LED_D3.0mm" (at 35.56 137.16 90)
+      (effects (font (size 1.27 1.27)) hide)
+    )
+    (property "Datasheet" "" (at 35.56 137.16 90)
+      (effects (font (size 1.27 1.27)) hide)
+    )
+    (property "LCSC#" "" (at 35.56 137.16 0)
+      (effects (font (size 1.27 1.27)) hide)
+    )
+    (pin "1")
+    (pin "2")
+    (instances
+      (project "Punainen insinööri"
+        (path "/e5ef43d6-cafc-424f-9222-4ed75d8d1dc6"
+          (reference "LED8") (unit 1)
+        )
+      )
+    )
+  )
   (symbol (lib_id "power:GND") (at 228.6 88.9 0) (unit 1)
     (in_bom yes) (on_board yes) (dnp no)
@@
         )
       )
+    )
+  )
+  (symbol (lib_id "Device:LED_Small") (at 45.72 137.16 270) (mirror x) (unit 1)
+    (in_bom yes) (on_board yes) (dnp no)
+    (property "Reference" "LED7" (at 48.26 137.16 0)
+      (effects (font (size 1.27 1.27)) hide)
+    )
+    (property "Value" "LED_Small" (at 48.26 137.0965 0)
+      (effects (font (size 1.27 1.27)) hide)
+    )
+    (property "Footprint" "LED_THT:LED_D3.0mm" (at 45.72 137.16 90)
+      (effects (font (size 1.27 1.27)) hide)
+    )
+    (property "Datasheet" "C2827254" (at 45.72 137.16 90)
+      (effects (font (size 1.27 1.27)) hide)
+    )
+    (property "LCSC#" "C84263" (at 45.72 137.16 0)
+      (effects (font (size 1.27 1.27)) hide)
+    )
+    (pin "1")
+    (pin "2")
+    (instances
+      (project "Punainen insinööri"
+        (path "/e5ef43d6-cafc-424f-9222-4ed75d8d1dc6"
+          (reference "LED7") (unit 1)
+        )
+      )
